Commit message: Add files via upload

File: drone/urdf/drone.urdf (robot description, URDF)
Before this commit: robot drone, 5 links, 4 joints
Links:
- link Motor1: mass 0.0055956 -> 0.00559561512965552
- link Motor2: mass 0.0055956 -> 0.00559561512965553
- link base_link: mass 0.49647 -> 0.496467844881593
Joints:
- joint Motor1_cont: origin xyz=0.38789 -0.21724 0.17864 rpy=1.5708 -1.5708 0 -> xyz=0.081 -0.251499999999997 0 rpy=0 0 0
- joint Motor2_cont: origin xyz=0.13639 -0.46874 0.17864 rpy=1.5708 -1.5708 0 -> xyz=0.0809999999999999 0 0.251499999999999 rpy=0 0 0
- joint Motor3_cont: origin xyz=0.13639 0.034256 0.17864 rpy=1.5708 -1.5708 0 -> xyz=0.081 0 -0.2515 rpy=0 0 0
- joint Motor4_cont: origin xyz=-0.11511 -0.21724 0.17864 rpy=1.5708 -1.5708 0 -> xyz=0.081 0.2515 0 rpy=0 0 0
